File: Hardware/LogBoard.brd (EAGLE design)
At the start: 34.3 x 48.3 mm, 54 parts, among them CN1 uSD Card, IC1 ESP12E, IC2 DS1391, IC3 FT232RQ, IC4 MAX14591, IC5 MAX14591, IC6 MAX1811, IC7 MAX8625, IC8 DS1722, X1 32.768k

Commit message: Updated Eagle PCB
Parts:
- SV2: device con-lstb:MA09-2 -> 000_Renan_Duarte:PH-9X2-180
Other:
- board text added: "Jump wire CD -> GPIO4"

Commit message: Updated BOM
Parts:
- C11, C4: value 10u/10V -> 1u/10V
- C12: value 0.33F/5.5V -> 100n/10V; device 000_Renan_Duarte:C-PTH-5X11.5 -> 000_Renan_Duarte:C-SMD-0603
- C13, C14: value 1u/10V -> 100n/10V
- C15: value 47u/6.3V -> 10u/10V; device rcl:CT3528 -> 000_Renan_Duarte:C-SMD-0603
- C16: value 47u6.3V -> 100n/10V; device rcl:CT3528 -> 000_Renan_Duarte:C-SMD-0603
- C2, C3: value 100n/10V -> 47u/6.3V; device 000_Renan_Duarte:C-SMD-0603 -> 000_Renan_Duarte:C-SMD-CT3528
- C5: value 100n/10V -> 1u/10V
- C6: value 1u/10V -> 0.33F/5.5V; device 000_Renan_Duarte:C-SMD-0603 -> 000_Renan_Duarte:C-PTH-5X11.5
- C7: value 100n/10V -> 10u/10V
- IC2: value DS1391 -> FT232RQ; device 000_Renan_Duarte:IC-USOP10 -> 000_Renan_Duarte:IC-QFN32
- IC3: value FT232RQ -> MAX14591ETA+; device 000_Renan_Duarte:IC-QFN32 -> 000_Renan_Duarte:IC-TDFN8
- IC4: value MAX14591 -> MAX14591ETA+
- IC5: value MAX14591 -> MAX1811ESA+; device 000_Renan_Duarte:IC-TDFN8 -> 000_Renan_Duarte:IC-SO8
- IC6: value MAX1811 -> MAX8625AETD+; device 000_Renan_Duarte:IC-SO8 -> 000_Renan_Duarte:IC-TDFN14
- IC7: value MAX8625 -> DS1391U-33+; device 000_Renan_Duarte:IC-TDFN14 -> 000_Renan_Duarte:IC-USOP10
- IC8: value DS1722 -> DS1722S+
- J1: value (none) -> C77238
- J2: value uSD Card -> THD2528-11SD-GF
- J3: value (none) -> HEADER 2x9 180
- Q1: value (none) -> BC847BS-7-F
- R1: value 0/WAKE -> 10k
- R10: value 1k -> 33
- R11: value 390k -> 33
- R12: value 100k -> 1k
- R13: value 10k -> 1k
- R2: value 10k -> 0/WAKE
- R3: value 10k -> 390k
- R4: value 10k -> 100k
- R7, R9: value 33 -> 10k
- R8: value 1k -> 10k
- S1: value POWER -> SK-3296S-01-L1
- S2: value RST -> TS24CA
- moved R11 39.8 mm to (11.4, 4.45), turned to 270 degrees
- moved R12 39.8 mm to (14.0, 4.45), turned to 270 degrees
- moved C3 33.3 mm to (9.21, 41.0), turned to 90 degrees
- moved C2 32.3 mm to (13.0, 41.0), turned to 90 degrees
- moved C14 28.2 mm to (1.59, 17.8), turned to 270 degrees
- moved R3 28.1 mm to (11.7, 44.3), turned to 180 degrees
- moved R4 28.1 mm to (14.3, 44.3), turned to 180 degrees
- moved IC2 25.3 mm to (5.40, 9.21)
- moved R7 24.9 mm to (30.8, 21.6), turned to 90 degrees
- moved C16 24.8 mm to (4.13, 17.8), turned to 270 degrees
- moved C15 24.0 mm to (2.86, 17.8), turned to 270 degrees
- moved R13 24.0 mm to (15.2, 4.45)
- moved R9 23.2 mm to (27.0, 21.6), turned to 90 degrees
- moved C4 23.0 mm to (29.5, 21.6)
- moved IC7 22.5 mm to (29.2, 17.8), turned to 0 degrees
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- renumbered BAT+ to PAD1, BAT- to PAD2, CN1 to J2, L3 to L1, SV2 to J3
Connections:
- net 3V3: now also C13.P$2, C15.P$1, C16.P$1, C2.+, C3.+, C4.P$1, C5.P$1, IC3.8, IC6.10, IC6.9, R1.P$2, R5.P$2, R7.P$2; no longer C10.P$1, C11.P$1, C13.P$1, C14.P$1, C15.+, C16.+, C8.P$2, IC2.10, IC5.8, IC7.9, R2.P$2, R3.P$2, R4.P$2
- net 3V3FTDI: now also C12.P$2, C8.P$2, IC2.1, IC2.16, IC2.18, IC3.4; no longer C3.P$2, C7.P$2, IC3.16, IC3.18, IC5.1, IC5.4
- net 5V0: now also C7.P$2, C9.P$2, IC2.19, IC5.2, IC5.4, IC5.7, R12.P$1, R13.P$2; no longer C2.P$2, C4.P$2, IC3.19, IC6.2, IC6.4, IC6.7, R10.P$2, R8.P$1
- net DTR: now also IC4.7, R9.P$2; no longer IC5.7, R6.P$2
- net FTDI_DTR: now also IC2.31, IC4.2; no longer IC3.31, IC5.2
- net FTDI_RTS: now also IC2.32, IC3.3; no longer IC3.32, IC4.3
- net FTDI_RX: now also IC2.2; no longer IC4.2
- net FTDI_TX: now also IC2.30, IC4.3; no longer IC3.30, IC5.3
- net GND: now also C12.P$1, C13.P$1, C15.P$2, C16.P$2, C2.-, C3.-, C4.P$2, C6.N, C9.P$1, IC2.17, IC2.20, IC2.24, IC2.26, IC2.4, IC2.GND, IC3.5, IC5.3, IC5.6, IC6.11, IC6.12, IC6.7, IC6.TP, IC7.5, R4.P$1, R6.P$1; no longer C12.N, C13.P$2, C15.-, C16.-, C2.P$1, C3.P$1, C4.P$1, C6.P$2, C9.P$2, IC2.5, IC3.17, IC3.20, IC3.24, IC3.26, IC3.4, IC3.GND, IC5.5, IC6.3, IC7.11, IC7.12, IC7.6, IC7.7, IC7.TP, R12.P$1, R13.P$1
- net GPIO0: now also R5.P$1; no longer R3.P$1
- net GPIO1/TX: now also IC3.7; no longer IC4.7
- net GPIO10/CSRTC: now also IC7.4; no longer IC2.4
- net GPIO12/MISO: now also IC7.7; no longer IC2.7
- net GPIO13/MOSI: now also IC7.6; no longer IC2.6
- net GPIO14/CLK: now also IC7.8; no longer IC2.8
- net GPIO15: now also R6.P$2; no longer R13.P$2
- net GPIO16: now also R2.P$1; no longer R1.P$1
- net GPIO2/INTRTC: now also IC7.9, R7.P$1; no longer IC2.9, R4.P$1
- net GPIO3/RX: now also IC4.6; no longer IC5.6
- net LED_CHG: now also IC5.8; no longer IC6.8
- net LED_RX: now also IC2.21, R11.P$1; no longer IC3.21, R9.P$1
- net LED_TX: now also IC2.22, R10.P$1; no longer IC3.22, R7.P$1
- net N$1: now also R8.P$1; no longer R5.P$1
- net N$10: now also IC5.1; no longer IC6.1
- net N$11: now also IC6.1, IC6.2; no longer IC7.1, IC7.2
- net N$16: now also IC6.3, IC6.4; no longer IC7.3, IC7.4
- net N$17: now also R3.P$1, R4.P$2; no longer R11.P$1, R12.P$2
- net N$18: now also IC7.1; no longer IC2.1
- net N$19: now also IC7.2; no longer IC2.2
- net N$2: now also R9.P$1; no longer R6.P$1
- net N$20: now also C14.P$1, IC6.8; no longer C9.P$1, IC7.8
- net N$22: now also R13.P$1; no longer R10.P$1
- net N$4: now also IC2.15; no longer IC3.15
- net N$5: now also IC2.14; no longer IC3.14
- net N$6: now also R10.P$2; no longer R7.P$2
- net N$7: now also R11.P$2; no longer R9.P$2
- net N$8: now also R12.P$2; no longer R8.P$2
- net PWRON: now also IC6.5; no longer IC7.5
- net RST: now also R1.P$1, R2.P$2; no longer R1.P$2, R2.P$1
- net RTS: now also IC3.6, R8.P$2; no longer IC4.6, R5.P$2
- net VBAT: now also C10.P$1, C11.P$1, IC5.5, IC6.13, IC6.14, R3.P$2; no longer C5.P$1, C6.P$1, IC6.5, IC7.13, IC7.14, R11.P$2
- net VBKP: now also C6.P, IC7.3; no longer C12.P, IC2.3
